Commit message: update

File: onrobotsg_description/urdf/sga/onrobotsg_a_macro.urdf.xacro (robot description, xacro)
@@ -8,16 +8,7 @@
 		</joint>
 		<link name="${prefix}onrobotsg_base_link">
-			<!-- <visual>
-				<origin xyz="0 0 0" rpy="0 0 0" />
-				<geometry>
-					<sphere radius="0.007"/>
-				</geometry>
-				<material name="">
-					<color rgba="0 1.0 0 1.0"/>
-				</material>
-			</visual> -->
 			<visual> <!-- Gripper body -->
 				<geometry>
-					<mesh filename="package://onrobotsg_description/meshes/visual/sga_full.STL"
+					<mesh filename="package://aljnump_description/meshes/sg/visual/sga_full.STL"
 						scale="0.001 0.001 0.001" />
 				</geometry>
@@ -25,5 +16,5 @@
 			<collision>
 				<geometry>
-					<mesh filename="package://onrobotsg_description/meshes/collision/plate_and_hub.STL"
+					<mesh filename="package://aljnump_description/meshes/sg/collision/plate_and_hub.STL"
 						scale="0.001 0.001 0.001" />
 				</geometry>
@@ -37,4 +28,20 @@
 			</inertial>
 		</link>
+		<link name="${prefix}onrobotsg_tip">
+			<visual>
+				<origin xyz="0 0 0" rpy="0 0 0" />
+				<geometry>
+					<sphere radius="0.007"/>
+				</geometry>
+				<material name="">
+					<color rgba="0 1.0 0 1.0"/>
+				</material>
+			</visual>
+		</link>
+		<joint name="${prefix}onrobotsg_base_tip_joint" type="fixed">
+			<parent link="${prefix}onrobotsg_base_link"/>
+			<child link="${prefix}onrobotsg_tip"/>
+			<origin xyz="0 0 0.15" rpy="0 0 0"/>
+		</joint>
 	</xacro:macro>
 </robot>

File: onrobotsg_description/urdf/sgb/onrobotsg_b_macro.urdf.xacro (robot description, xacro)
@@ -8,16 +8,7 @@
 		</joint>
 		<link name="${prefix}onrobotsg_base_link">
-			<!-- <visual>
-				<origin xyz="0 0 0" rpy="0 0 0" />
-				<geometry>
-					<sphere radius="0.007"/>
-				</geometry>
-				<material name="">
-					<color rgba="0 1.0 0 1.0"/>
-				</material>
-			</visual> -->
 			<visual> <!-- Gripper body -->
 				<geometry>
-					<mesh filename="package://onrobotsg_description/meshes/visual/sgb_full.STL"
+					<mesh filename="package://aljnump_description/meshes/sg/visual/sgb_full.STL"
 						scale="0.001 0.001 0.001" />
 				</geometry>
@@ -25,5 +16,5 @@
 			<collision>
 				<geometry>
-					<mesh filename="package://onrobotsg_description/meshes/collision/plate_and_hub.STL"
+					<mesh filename="package://aljnump_description/meshes/sg/collision/plate_and_hub.STL"
 						scale="0.001 0.001 0.001" />
 				</geometry>
@@ -37,4 +28,20 @@
 			</inertial>
 		</link>
+		<link name="${prefix}onrobotsg_tip">
+			<visual>
+				<origin xyz="0 0 0" rpy="0 0 0" />
+				<geometry>
+					<sphere radius="0.007"/>
+				</geometry>
+				<material name="">
+					<color rgba="0 1.0 0 1.0"/>
+				</material>
+			</visual>
+		</link>
+		<joint name="${prefix}onrobotsg_base_tip_joint" type="fixed">
+			<parent link="${prefix}onrobotsg_base_link"/>
+			<child link="${prefix}onrobotsg_tip"/>
+			<origin xyz="0 0 0.15" rpy="0 0 0"/>
+		</joint>
 	</xacro:macro>
 </robot>

Commit message: update

File: onrobotsg_description/urdf/sga/onrobotsg_a_macro.urdf.xacro (robot description, xacro)
@@ -10,5 +10,5 @@
 			<visual> <!-- Gripper body -->
 				<geometry>
-					<mesh filename="package://aljnump_description/meshes/sg/visual/sga_full.STL"
+					<mesh filename="package://onrobotsg_description/meshes/sg/visual/sga_full.STL"
 						scale="0.001 0.001 0.001" />
 				</geometry>
@@ -16,5 +16,5 @@
 			<collision>
 				<geometry>
-					<mesh filename="package://aljnump_description/meshes/sg/collision/plate_and_hub.STL"
+					<mesh filename="package://onrobotsg_description/meshes/sg/collision/plate_and_hub.STL"
 						scale="0.001 0.001 0.001" />
 				</geometry>

File: onrobotsg_description/urdf/sgb/onrobotsg_b_macro.urdf.xacro (robot description, xacro)
@@ -10,5 +10,5 @@
 			<visual> <!-- Gripper body -->
 				<geometry>
-					<mesh filename="package://aljnump_description/meshes/sg/visual/sgb_full.STL"
+					<mesh filename="package://onrobotsg_description/meshes/sg/visual/sgb_full.STL"
 						scale="0.001 0.001 0.001" />
 				</geometry>
@@ -16,5 +16,5 @@
 			<collision>
 				<geometry>
-					<mesh filename="package://aljnump_description/meshes/sg/collision/plate_and_hub.STL"
+					<mesh filename="package://onrobotsg_description/meshes/sg/collision/plate_and_hub.STL"
 						scale="0.001 0.001 0.001" />
 				</geometry>

Commit message: update

File: onrobotsg_description/urdf/sga/onrobotsg_a_macro.urdf.xacro (robot description, xacro)
@@ -10,5 +10,5 @@
 			<visual> <!-- Gripper body -->
 				<geometry>
-					<mesh filename="package://onrobotsg_description/meshes/sg/visual/sga_full.STL"
+					<mesh filename="package://onrobotsg_description/meshes/visual/sga_full.STL"
 						scale="0.001 0.001 0.001" />
 				</geometry>
@@ -16,5 +16,5 @@
 			<collision>
 				<geometry>
-					<mesh filename="package://onrobotsg_description/meshes/sg/collision/plate_and_hub.STL"
+					<mesh filename="package://onrobotsg_description/meshes/collision/plate_and_hub.STL"
 						scale="0.001 0.001 0.001" />
 				</geometry>

File: onrobotsg_description/urdf/sgb/onrobotsg_b_macro.urdf.xacro (robot description, xacro)
@@ -10,5 +10,5 @@
 			<visual> <!-- Gripper body -->
 				<geometry>
-					<mesh filename="package://onrobotsg_description/meshes/sg/visual/sgb_full.STL"
+					<mesh filename="package://onrobotsg_description/meshes/visual/sgb_full.STL"
 						scale="0.001 0.001 0.001" />
 				</geometry>
@@ -16,5 +16,5 @@
 			<collision>
 				<geometry>
-					<mesh filename="package://onrobotsg_description/meshes/sg/collision/plate_and_hub.STL"
+					<mesh filename="package://onrobotsg_description/meshes/collision/plate_and_hub.STL"
 						scale="0.001 0.001 0.001" />
 				</geometry>
